Commit message: demo trajectories

File: examples/box0.urdf (robot description, URDF)
Before this commit: robot block_2, 1 links, 0 joints
Links:
- link block_2_base_link: geometry collision box size=0.0 0.0 0.0; visual box size=0.2 1.75 1

File: examples/box3.urdf (robot description, URDF)
Before this commit: robot block_2, 1 links, 0 joints
Links:
- link block_2_base_link: geometry collision box size=0.0 0.0 0.0; visual box size=0.09999999999999998 0.09999999999999998 1

File: examples/box4.urdf (robot description, URDF)
Before this commit: robot block_2, 1 links, 0 joints
Links:
- link block_2_base_link: geometry collision box size=0.0 0.0 0.0; visual box size=0.09999999999999998 0.10000000000000003 1
